Commit message: gazebo 环境完成

File: src/sunny_gazebo/urdf/sunny_model.gazebo.xacro (robot description, xacro)
@@ -105,4 +105,36 @@
     </sensor>
   </gazebo>
+  <gazebo reference="top_laser_link">
+    <material>Gazebo/FlatBlack</material>
+    <sensor type="ray" name="top_lds_lfcd_sensor">
+      <pose>0 0 0 0 0 0</pose>
+      <visualize>false</visualize>
+      <update_rate>10</update_rate>
+      <ray>
+        <scan>
+          <horizontal>
+            <samples>361</samples>
+            <resolution>1</resolution>
+            <min_angle>-${180*M_PI/180}</min_angle>
+            <max_angle>${180*M_PI/180}</max_angle>
+          </horizontal>
+        </scan>
+        <range>
+          <min>0.1</min>
+          <max>8</max>
+          <resolution>0.01</resolution>
+        </range>
+        <noise>
+          <type>gaussian</type>
+          <mean>0.0</mean>
+          <stddev>0.01</stddev>
+        </noise>
+      </ray>
+      <plugin name="gazebo_ros_lds_lfcd_controller" filename="libgazebo_ros_laser.so">
+        <topicName>top_scan</topicName>
+        <frameName>top_laser_link</frameName>
+      </plugin>
+    </sensor>
+  </gazebo>
   <!-- <gazebo reference="bumper_link">
     <sensor name="bumper" type="contact">

File: src/sunny_gazebo/urdf/sunny_model.urdf.xacro (robot description, xacro)
@@ -340,4 +340,20 @@
       k_velocity="0" />
   </joint>
+  <link name="top_laser_link"/>
+  <joint
+    name="top_joint_ladar"
+    type="fixed">
+    <origin
+      xyz="0.0 0 2.0"
+      rpy="0 0 0" />
+    <parent
+      link="base_link" />
+    <child
+      link="top_laser_link" />
+    <axis
+      xyz="0 0 0" />
+    <safety_controller
+      k_velocity="0" />
+  </joint>
   <!--Ultrasonic (TBD) -->
   <!-- <link name="bumper_link">
